Commit message: Add transmission property
J joints are revolute,  wheel joints are continous
J joints use effort controller, wheel joints use velocity controller

File: urdf/newbot2.urdf (robot description, URDF)
Before this commit: robot newbot2, 10 links, 9 joints
Joints:
- joint FL_J: limit (none) -> lower=-1 upper=1 effort=10.0 velocity=0.5; type continuous -> revolute
- joint FR_J: limit (none) -> lower=-1 upper=1 effort=10.0 velocity=0.5; type continuous -> revolute

Commit message: Add controller for 4 Wheels
4 Wheels use jointgroupvelocity control
Adjust the pid value of controllers
the dynamic fiction has to be < 1 to move

File: urdf/newbot2.urdf (robot description, URDF)
Before this commit: robot newbot2, 10 links, 9 joints
Links:
- removed link world
- added link dummy
Joints:
- removed joint world_J
- added joint dummy: type fixed, parent dummy, child base_link
- joint FL_J: limit lower=-1 upper=1 effort=10.0 velocity=0.5 -> lower=-1 upper=1 effort=100.0 velocity=10
- joint FR_J: limit lower=-1 upper=1 effort=10.0 velocity=0.5 -> lower=-1 upper=1 effort=100.0 velocity=10
- joint WFL_J: limit (none) -> effort=100.0 velocity=10
- joint WFR_J: limit (none) -> effort=100.0 velocity=10
- joint WRL_J: limit (none) -> effort=100.0 velocity=10
- joint WRR_J: limit (none) -> effort=100.0 velocity=10

Commit message: Fix rear wheels free rolling problem
The rear wheels has to use the joint_state_controller through
extra_joints for rviz to get the correct tf reading.

File: urdf/newbot2.urdf (robot description, URDF)
Before this commit: robot newbot2, 10 links, 9 joints
Joints:
- joint FL_J: limit lower=-1 upper=1 effort=100.0 velocity=10 -> lower=-1 upper=1 effort=100.0 velocity=30
- joint FR_J: limit lower=-1 upper=1 effort=100.0 velocity=10 -> lower=-1 upper=1 effort=100.0 velocity=30

Commit message: Add lidar sensor
todo: the lidar visual position correction

File: urdf/newbot2.urdf (robot description, URDF)
Before this commit: robot newbot2, 10 links, 9 joints
Links:
- added link Lidar_L, mass 0.0730843684055266; collision mesh filename=package://newbot2/meshes/Lidar_L.STL; visual mesh filename=package://newbot2/meshes/Lidar_L.STL
Joints:
- added joint Lidar_J: type fixed, parent base_link, child Lidar_L, origin xyz=0 0 0.3 rpy=0 0 0, axis 0 0 1

Commit message: Fix lidar position

File: urdf/newbot2.urdf (robot description, URDF)
Before this commit: robot newbot2, 11 links, 10 joints
Joints:
- joint Lidar_J: axis 0 0 1 -> 0 0 0; origin xyz=0 0 0.3 rpy=0 0 0 -> xyz=0 0 0.28597 rpy=0 0 0

Commit message: Adjust bot speed param

File: urdf/newbot2.urdf (robot description, URDF)
Before this commit: robot newbot2, 11 links, 10 joints
Joints:
- joint WFL_J: limit effort=100.0 velocity=10 -> effort=100.0 velocity=50
- joint WFR_J: limit effort=100.0 velocity=10 -> effort=100.0 velocity=50
- joint WRL_J: limit effort=100.0 velocity=10 -> effort=100.0 velocity=50
- joint WRR_J: limit effort=100.0 velocity=10 -> effort=100.0 velocity=50
